Commit message: collisions, draw environment

File: wxai_draw.urdf (robot description, URDF)
Before this commit: robot wxai, 15 links, 14 joints
Links:
- removed link ee_gripper_link
- added link pen_link, mass 0.001; collision cylinder length=0.08 radius=0.01; visual cylinder length=0.08 radius=0.01
- added link pen_tip_link, mass 0.0001; collision sphere radius=0.005; visual sphere radius=0.005
- link camera_bottom_screw_frame: mass None -> 0.001
Joints:
- removed joint ee_gripper
- added joint pen: type fixed, parent link_6, child pen_link, origin xyz=0.142 0 0 rpy=0 -0.78539816339 0, axis 1 0 0
- added joint pen_tip_joint: type fixed, parent pen_link, child pen_tip_link, origin xyz=0 0 -0.04 rpy=0 0 0
